File: LM5160.kicad_pcb (KiCad board)
At the start: 4 copper layers, 48.3 x 17.8 mm, 70 parts, among them J1 Analog, J2 Digital, J3 SolderJumper_2_Open, J4 VOUT, J5 VIN, U1 LM5160DNTR

Commit message: Add files via upload
Parts:
- moved SYM4 192.5 mm to (4.20, -12.8)
- moved R8 10.5 mm to (20.6, -20.6)
- moved TP13 8.42 mm to (21.6, -3.45)
- moved D5 8.40 mm to (24.5, -20.1)
- moved TP15 7.33 mm to (7.35, -5.40)
- moved TP7 5.51 mm to (27.1, -3.65)
- moved C12 5.36 mm to (23.8, -8.10), turned to -90 degrees
- moved R7 5.31 mm to (23.8, -11.1), turned to 90 degrees
- moved C13 4.41 mm to (25.3, -11.1), turned to 90 degrees
- moved TP17 3.60 mm to (12.2, -9.25)
- moved R11 3.24 mm to (22.3, -8.10), turned to -90 degrees
- moved TP10 3.06 mm to (20.1, -5.10)
- moved FID2 2.61 mm to (15.2, -3.20)
- moved C11 2.50 mm to (15.6, -6.65)
- moved R12 2.47 mm to (25.3, -8.10), turned to -90 degrees
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Routing:
- net /VIN: track 2.78 -> 19.9 mm
- net GNDREF: track 5.67 -> 12.3 mm, vias 0 -> 1
- net /VCCIC: track 0.00 -> 6.11 mm
- net /SS: track 0.00 -> 5.61 mm
- net /EN: track 0.00 -> 4.94 mm
- net /RON: track 0.00 -> 4.54 mm
- net Net-(D4-A): track 0.00 -> 1.39 mm

Commit message: Add files via upload
Parts:
- C1, C3, C4: footprint Capacitor_SMD:C_1206_3216Metric -> LM5160:C_1206_3216Metric
- C10, C11, C12, C13, C14, C15, C2, C5, C6, C8: footprint Capacitor_SMD:C_0603_1608Metric -> LM5160:C_0603_1608Metric
- C7: footprint Capacitor_SMD:C_0805_2012Metric -> LM5160:C_0805_2012Metric
- D1, D4, D5: footprint LED_SMD:LED_0603_1608Metric -> LM5160:LED_0603_1608Metric
- D2: footprint Diode_SMD:D_SOD-123F -> LM5160:D_SOD-123F
- FID1, FID2, FID3: footprint Fiducial:Fiducial_0.75mm_Mask2.25mm -> LM5160:Fiducial_0.75mm_Mask2.25mm
- J1, J2: footprint Connector_PinHeader_2.54mm:PinHeader_1x17_P2.54mm_Vertical -> LM5160:PinHeader_1x17_P2.54mm_Vertical
- J3: footprint Jumper:SolderJumper-2_P1.3mm_Open_Pad1.0x1.5mm -> LM5160:SolderJumper-2_P1.3mm_Open_Pad1.0x1.5mm
- J4, J5: footprint Connector_PinHeader_2.54mm:PinHeader_1x02_P2.54mm_Vertical -> LM5160:PinHeader_1x02_P2.54mm_Vertical
- L1, L2: footprint Inductor_SMD:L_0603_1608Metric -> LM5160:L_0603_1608Metric
- MH1, MH2, MH3, MH4: footprint Arduino_MountingHole:MountingHole_1.2mm -> LM5160:MountingHole_1.2mm
- R1, R10, R11, R12, R13, R2, R3, R4, R5, R6, R7, R8, R9: footprint Resistor_SMD:R_0603_1608Metric -> LM5160:R_0603_1608Metric
- SYM1: footprint Symbol:OSHW-Symbol_6.7x6mm_SilkScreen -> LM5160:OSHW-Symbol_6.7x6mm_SilkScreen
- SYM2: footprint Symbol:ESD-Logo_6.6x6mm_SilkScreen -> LM5160:ESD-Logo_6.6x6mm_SilkScreen
- SYM3: footprint Symbol:WEEE-Logo_4.2x6mm_SilkScreen -> LM5160:WEEE-Logo_4.2x6mm_SilkScreen
- SYM4: footprint Symbol:LayerMarker_4_6.35x2.54mm_TextH1mm_P1.27mm_BottomMirrored -> LM5160:LayerMarker_4_6.35x2.54mm_TextH1mm_P1.27mm_BottomMirrored
- SYM5: footprint Symbol:KiCad-Logo2_5mm_SilkScreen -> LM5160:KiCad-Logo2_5mm_SilkScreen
- TP1, TP10, TP11, TP12, TP13, TP14, TP15, TP16, TP17, TP18, TP19, TP2, TP3, TP4, TP5, TP6, TP7, TP8, TP9: footprint TestPoint:TestPoint_Pad_D1.0mm -> LM5160:TestPoint_Pad_D1.0mm
- U1: footprint Package_SON:WSON-12-1EP_4x4mm_P0.5mm_EP2.6x3mm_ThermalVias -> LM5160:WSON-12-1EP_4x4mm_P0.5mm_EP2.6x3mm_ThermalVias
- moved FID3 1.30 mm to (46.1, -12.5)
Other:
- board text removed: "0"
- board text removed: "0 mils"
- board text removed: "0.02"
- board text removed: "0.3937 mils"
- board text removed: "1"
- board text removed: "1.37795 mils"
- board text removed: "11.81 mils"
- board text removed: "1900.00 mils x 700.00 mils"
- board text removed: "3.3"
- board text removed: "3.93701 mils"
- board text removed: "4"
- board text removed: "4.5"
- board text removed: "48.8189 mils"
- board text removed: "62.99 mils"
- board text removed: "7.87 mils / 0.00 mils"
- board text removed: "B.Cu"
- board text removed: "B.Mask"
- board text removed: "B.Paste"
- board text removed: "B.Silkscreen"
- board text removed: "BOARD CHARACTERISTICS"
- board text removed: "Board Thickness:"
- board text removed: "Board overall dimensions:"
- board text removed: "Bottom Silk Screen"
- board text removed: "Bottom Solder Mask"
- board text removed: "Bottom Solder Paste"
- board text removed: "Castellated pads:"
- board text removed: "Color"
- board text removed: "Copper Finish:"
- board text removed: "Copper Layer Count:"
- board text removed: "Dielectric 1"
- board text removed: "Dielectric 2"
- board text removed: "Dielectric 3"
- board text removed: "Edge card connectors:"
- board text removed: "Epsilon R"
- board text removed: "F.Cu"
- board text removed: "F.Mask"
- board text removed: "F.Paste"
- board text removed: "F.Silkscreen"
- board text removed: "FR4"
- board text removed: "FR4 natural"
- board text removed: "Green"
- board text removed: "Impedance Control:"
- board text removed: "In1.Cu"
- board text removed: "In2.Cu"
- board text removed: "Layer Name"
- board text removed: "Loss Tangent"
- board text removed: "Material"
- board text removed: "Min hole diameter:"
- board text removed: "Min track/spacing:"
- board text removed: "No"
- board text removed: "None"
- board text removed: "Not specified"
- board text removed: "Plated Board Edge:"
- board text removed: "Thickness (mils)"
- board text removed: "Top Silk Screen"
- board text removed: "Top Solder Mask"
- board text removed: "Top Solder Paste"
- board text removed: "Type"
- board text removed: "White"
- board text removed: "copper"
- board text removed: "core"
- board text removed: "prepreg"
