File: LM5160.kicad_sch (KiCad schematic)
At the start: 67 parts, among them J1 Analog, J2 Digital, J3 SolderJumper_2_Open, J4 VOUT, J5 VIN, U1 LM5160DNTR

Commit message: Add files via upload
Other:
- moved on the sheet: SYM1, SYM2, SYM3, SYM4, SYM5
Changed lines of the file:
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@@
 	(symbol
 		(lib_id "Graphic:Logo_Open_Hardware_Small")
-		(at 63.5 228.6 0)
+		(at 50.8 228.6 0)
 		(unit 1)
-		(exclude_from_sim no)
+		(exclude_from_sim yes)
 		(in_bom no)
 		(on_board yes)
@@
 		(fields_autoplaced yes)
 		(property "Reference" "SYM1"
-			(at 63.5 221.615 0)
+			(at 50.8 221.615 0)
 			(effects
 				(font
@@
 		)
 		(property "Value" "Logo_Open_Hardware_Small"
-			(at 63.5 234.315 0)
+			(at 50.8 234.315 0)
 			(effects
 				(font
@@
 		)
 		(property "Footprint" "Symbol:OSHW-Symbol_6.7x6mm_SilkScreen"
-			(at 63.5 228.6 0)
+			(at 50.8 228.6 0)
 			(effects
 				(font
@@
 		)
 		(property "Datasheet" "~"
-			(at 63.5 228.6 0)
+			(at 50.8 228.6 0)
 			(effects
 				(font
@@
 		)
 		(property "Description" "Open Hardware logo, small"
-			(at 63.5 228.6 0)
-			(effects
-				(font
-					(size 1.27 1.27)
-				)
-				(hide yes)
-			)
-		)
-		(property "Sim.Enable" "0"
-			(at 63.5 228.6 0)
+			(at 50.8 228.6 0)
 			(effects
 				(font
@@
 	(symbol
 		(lib_id "Mechanical:Fiducial")
-		(at 114.3 228.6 0)
+		(at 101.6 228.6 0)
 		(unit 1)
 		(exclude_from_sim no)
@@
 		(fields_autoplaced yes)
 		(property "Reference" "SYM3"
-			(at 116.84 227.3299 0)
+			(at 104.14 227.3299 0)
 			(effects
 				(font
@@
 		)
 		(property "Value" "WEEE"
-			(at 116.84 229.8699 0)
+			(at 104.14 229.8699 0)
 			(effects
 				(font
@@
 		)
 		(property "Footprint" "Symbol:WEEE-Logo_4.2x6mm_SilkScreen"
-			(at 114.3 228.6 0)
+			(at 101.6 228.6 0)
 			(effects
 				(font
@@
 		)
 		(property "Datasheet" "~"
-			(at 114.3 228.6 0)
+			(at 101.6 228.6 0)
 			(effects
 				(font
@@
 		)
 		(property "Description" "Fiducial Marker"
-			(at 114.3 228.6 0)
+			(at 101.6 228.6 0)
 			(effects
 				(font
@@
 	(symbol
 		(lib_id "Mechanical:Fiducial")
-		(at 114.3 236.22 0)
+		(at 114.3 228.6 0)
 		(unit 1)
 		(exclude_from_sim no)
@@
 		(fields_autoplaced yes)
 		(property "Reference" "SYM4"
-			(at 116.84 234.9499 0)
+			(at 116.84 227.3299 0)
 			(effects
 				(font
@@
 		)
 		(property "Value" "LAYERS"
-			(at 116.84 237.4899 0)
+			(at 116.84 229.8699 0)
 			(effects
 				(font
@@
 		)
 		(property "Footprint" "Symbol:LayerMarker_4_6.35x2.54mm_TextH1mm_P1.27mm_BottomMirrored"
-			(at 114.3 236.22 0)
+			(at 114.3 228.6 0)
 			(effects
 				(font
@@
 		)
 		(property "Datasheet" "~"
-			(at 114.3 236.22 0)
+			(at 114.3 228.6 0)
 			(effects
 				(font
@@
 		)
 		(property "Description" "Fiducial Marker"
-			(at 114.3 236.22 0)
+			(at 114.3 228.6 0)
 			(effects
 				(font
@@
 	(symbol
 		(lib_id "Graphic:SYM_ESD_Large")
-		(at 88.9 228.6 0)
+		(at 76.2 227.33 0)
 		(unit 1)
-		(exclude_from_sim no)
+		(exclude_from_sim yes)
 		(in_bom no)
 		(on_board yes)
@@
 		(fields_autoplaced yes)
 		(property "Reference" "SYM2"
-			(at 88.9 223.52 0)
+			(at 76.2 222.25 0)
 			(effects
 				(font
@@
 		)
 		(property "Value" "SYM_ESD_Large"
-			(at 88.9 234.95 0)
+			(at 76.2 233.68 0)
 			(effects
 				(font
@@
 		)
 		(property "Footprint" "Symbol:ESD-Logo_6.6x6mm_SilkScreen"
-			(at 88.773 229.362 0)
+			(at 76.073 228.092 0)
 			(effects
 				(font
@@
 		)
 		(property "Datasheet" "~"
-			(at 88.773 229.362 0)
+			(at 76.073 228.092 0)
 			(effects
 				(font
@@
 		)
 		(property "Description" "ESD warning/\"Do not touch\" symbol, large"
-			(at 88.9 228.6 0)
-			(effects
-				(font
-					(size 1.27 1.27)
-				)
-				(hide yes)
-			)
-		)
-		(property "Sim.Enable" "0"
-			(at 88.9 228.6 0)
+			(at 76.2 227.33 0)
 			(effects
 				(font
@@
 	(symbol
 		(lib_id "Mechanical:Fiducial")
-		(at 114.3 243.84 0)
+		(at 127 228.6 0)
 		(unit 1)
 		(exclude_from_sim no)
@@
 		(fields_autoplaced yes)
 		(property "Reference" "SYM5"
-			(at 116.84 242.5699 0)
+			(at 129.54 227.3299 0)
 			(effects
 				(font
@@
 		)
 		(property "Value" "KICAD"
-			(at 116.84 245.1099 0)
+			(at 129.54 229.8699 0)
 			(effects
 				(font
@@
 		)
 		(property "Footprint" "KiCad-Logo2_5mm_SilkScreen"
-			(at 114.3 243.84 0)
+			(at 127 228.6 0)
 			(effects
 				(font
@@
 		)
 		(property "Datasheet" "~"
-			(at 114.3 243.84 0)
+			(at 127 228.6 0)
 			(effects
 				(font
@@
 		)
 		(property "Description" "Fiducial Marker"
-			(at 114.3 243.84 0)
+			(at 127 228.6 0)
 			(effects
 				(font
